Commit message: 4.0 - Motion Planning using Cpp - no message from topic /joint_states

File: myworkcell_support/urdf/workcell.urdf.xacro (robot description, xacro)
@@ -1,44 +1,44 @@
-<?xml version="1.0"?>
+<?xml version="1.0" ?>
 <robot name="myworkcell" xmlns:xacro="http://ros.org/wiki/xacro">
-  <link name="world" />
+  <xacro:include filename="$(find ur_description)/urdf/ur_macro.xacro"/>
+  <!-- ur arm instantiation -->
+  <xacro:arg name="ur_type" default="ur5"/>
+  <xacro:arg name="use_fake_hardware" default="true"/>
+  <xacro:arg name="fake_sensor_commands" default="true"/>
+  <xacro:ur_robot
+      name="my_ur5"
+      tf_prefix=""
+      parent="table"
+      joint_limits_parameters_file="$(find ur_description)/config/$(arg ur_type)/joint_limits.yaml"
+      kinematics_parameters_file="$(find ur_description)/config/$(arg ur_type)/default_kinematics.yaml"
+      physical_parameters_file="$(find ur_description)/config/$(arg ur_type)/physical_parameters.yaml"
+      visual_parameters_file="$(find ur_description)/config/$(arg ur_type)/visual_parameters.yaml"
+      use_fake_hardware="$(arg use_fake_hardware)"
+      fake_sensor_commands="$(arg fake_sensor_commands)">
+    <origin xyz="0 0 0" rpy="0 0 0"/>
+  </xacro:ur_robot>
+  <link name="world"/>
   <link name="table">
     <visual>
       <geometry>
-        <box size="1.0 1.0 0.05" />
+        <box size="1.0 1.0 0.05"/>
       </geometry>
     </visual>
     <collision>
       <geometry>
-        <box size="1.0 1.0 0.05" />
+        <box size="1.0 1.0 0.05"/>
       </geometry>
     </collision>
   </link>
-  <link name="camera_frame" />
-  <xacro:include filename="$(find ur_description)/urdf/ur_macro.xacro" />
-  <!-- ur arm instantiation -->
-  <xacro:arg name="ur_type" default="ur5" />
-  <xacro:arg name="use_fake_hardware" default="true" />
-  <xacro:arg name="fake_sensor_commands" default="true" />
-  <xacro:ur_robot
-    name="my_ur5"
-    tf_prefix=""
-    parent="table"
-    joint_limits_parameters_file="$(find ur_description)/config/$(arg ur_type)/joint_limits.yaml"
-    kinematics_parameters_file="$(find ur_description)/config/$(arg ur_type)/default_kinematics.yaml"
-    physical_parameters_file="$(find ur_description)/config/$(arg ur_type)/physical_parameters.yaml"
-    visual_parameters_file="$(find ur_description)/config/$(arg ur_type)/visual_parameters.yaml"
-    use_fake_hardware="$(arg use_fake_hardware)"
-    fake_sensor_commands="$(arg fake_sensor_commands)">
-    <origin xyz="0 0 0" rpy="0 0 0" /> // make the robot base link connect to our table link without any offset or rotation
-  </xacro:ur_robot>
+  <link name="camera_frame"/>
   <joint name="world_to_table" type="fixed">
-    <parent link="world" />
-    <child link="table" />
-    <origin xyz="0 0 0.5" rpy="0 0 0" />
+    <parent link="world"/>
+    <child link="table"/>
+    <origin xyz="0 0 0.5" rpy="0 0 0"/>
   </joint>
   <joint name="world_to_camera" type="fixed">
-    <parent link="world" />
-    <child link="camera_frame" />
-    <origin xyz="-0.25 -0.5 1.25" rpy="0 3.14159 0" />
+    <parent link="world"/>
+    <child link="camera_frame"/>
+    <origin xyz="-0.25 -0.5 1.25" rpy="0 3.14159 0"/>
   </joint>
 </robot>
